File: right/mpm62-kb-right.sch (KiCad schematic (older format))
At the start: 71 parts, among them J1 Conn_01x04_Male, J2 Conn_01x02_Male, U1 MCP23018-E_SP

Commit message: Final for b1t (board 1 thruhole) board
Parts:
- removed J2: Conn_01x02_Male, Connector_PinHeader_2.54mm:PinHeader_1x02_P2.54mm_Vertical, symbol Connector:Conn_01x02_Male
- added H1, H2, H3, H4: MountingHole, MountingHole:MountingHole_2.2mm_M2_Pad, symbol Mechanical:MountingHole
- added J2: JST ZH Header, MpmMisc:JST_ZH_B4B-ZR_1x04_P1.50mm_Vertical, symbol Connector:Conn_01x04_Male
- added U2: TRRS, Keebio-Parts:TRRS-PJ-320A, symbol keebio:TRRS
- J1: value Conn_01x04_Male -> Raw Header
- MX1, MX10, MX12, MX13, MX14, MX15, MX16, MX17, MX18, MX19, MX2, MX21, MX22, MX23, MX24, MX26, MX27, MX3, MX4, MX5, MX6, MX7, MX8, MX9: footprint MX_Alps_Hybrid:MX-1U-NoLED -> MX_Only:MXOnly-1U-NoLED
- MX11: footprint MX_Alps_Hybrid:MX-3U-ReversedStabilizers-NoLED -> MX_Only:MXOnly-3U-ReversedStabilizers-NoLED
- MX20, MX25, MX28, MX33: footprint MX_Alps_Hybrid:MX-1.25U-NoLED -> MX_Only:MXOnly-1.25U-NoLED
- MX29: footprint MX_Alps_Hybrid:MX-2U-NoLED -> MX_Only:MXOnly-2U-NoLED
- MX30: footprint MX_Alps_Hybrid:MX-1.5U-NoLED -> MX_Only:MXOnly-1.5U-NoLED
- MX31: footprint MX_Alps_Hybrid:MX-2.25U-NoLED -> MX_Only:MXOnly-2.25U-NoLED
- MX32: footprint MX_Alps_Hybrid:MX-2.75U-NoLED -> MX_Only:MXOnly-2.75U-NoLED
Connections:
- wire segments 122 -> 134
